Commit message: GPS at 2 Hz via a custom navsat xacro instead of stock garmin_18x
Clearpath's garmin_18x.urdf.xacro hardcodes <update_rate>1</update_rate>
and its macro takes only name/parent_link/origin, so the rate cannot be
raised from robot_configs/ — clearpath_config's GPS types carry no
update_rate field at all (only IMU does), and the generator emits
<xacro:garmin_18x name="gps_0" parent_link="sensor_arch_mount"> with no
rate argument. The vendor file must not be edited, so gps_0 is now a
custom sensor: urdf/gps_2hz.urdf.xacro, a copy of the vendor macro with
update_rate 2, instantiated from urdf/extras_default.urdf.xacro at the
same mount (sensor_arch_mount, xyz 0.0 0.15 0.0) and the same gz topic
(.../sensors/gps_0/navsat), bridged explicitly in run_husky_sim.sh with
a remap onto /a200_0000/sensors/gps_0/fix so the ROS topic is unchanged.

Verified in the generated SDF for both configs: gps_0 -> navsat with
update_rate 2 and pose 0 0.15 0.524, identical to the stock placement.

2 Hz is the user's decision, overriding the 10 Hz in §3.2 of
docs/superpowers/specs/2026-08-26-park-localization-revision-design.md;
that spec line is updated to match.

Co-Authored-By: Claude Opus 5 (1M context) <noreply@anthropic.com>
Claude-Session: https://claude.ai/code/session_01JDi76LXhp6hUJPewtxpvvX

File: urdf/extras_default.urdf.xacro (robot description, xacro)
@@ -5,3 +5,12 @@
   <xacro:include filename="/home/thinhpham/Documents/Husky_viz/urdf/wheel_slip.urdf.xacro"/>
   <xacro:include filename="/home/thinhpham/Documents/Husky_viz/urdf/imu_enu.urdf.xacro"/>
+  <xacro:include filename="/home/thinhpham/Documents/Husky_viz/urdf/gps_2hz.urdf.xacro"/>
+  <!-- Replaces the stock garmin_18x gps_0, which is locked to 1 Hz (its macro
+       takes no update_rate and the generator passes none). Same name, same
+       mount as the removed robot_configs/ entry, so the ROS topic is
+       unchanged: /a200_0000/sensors/gps_0/fix. Because it is a custom sensor
+       the mount has to live here rather than in robot_configs/. -->
+  <xacro:gps_2hz name="gps_0" parent_link="sensor_arch_mount">
+    <origin xyz="0.0 0.15 0.0" rpy="0.0 0.0 0.0"/>
+  </xacro:gps_2hz>
 </robot>
